File: hardware/jc-playstation/JC-Playstation.kicad_sch (KiCad schematic)
At the start: 18 parts, among them J1 JAMMACON, SW1 RESET, SW2 Analog-Digital, U1 ATmega328P-P, U2 ATmega328P-P, U3 7407, X1 PLAYER 1, X2 PLAYER 2

Commit message: Add files via upload
Changed lines of the file:
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@@
+    (stroke (width 0) (type default) (color 0 0 0 0))
+  )
+  (wire (pts (xy 273.05 154.94) (xy 273.05 158.75))
     (stroke (width 0) (type default) (color 0 0 0 0))
   )
@@
   )
   (wire (pts (xy 128.27 86.36) (xy 134.62 86.36))
+    (stroke (width 0) (type default) (color 0 0 0 0))
+  )
+  (wire (pts (xy 262.89 154.94) (xy 262.89 158.75))
     (stroke (width 0) (type default) (color 0 0 0 0))
   )
@@
     (pin "1")
   )
+  (symbol (lib_id "power:GND") (at 262.89 158.75 0) (unit 1)
+    (in_bom yes) (on_board yes) (fields_autoplaced)
+    (property "Reference" "#PWR05" (id 0) (at 262.89 165.1 0)
+      (effects (font (size 1.27 1.27)) hide)
+    )
+    (property "Value" "GND" (id 1) (at 262.89 163.83 0))
+    (property "Footprint" "" (id 2) (at 262.89 158.75 0)
+      (effects (font (size 1.27 1.27)) hide)
+    )
+    (property "Datasheet" "" (id 3) (at 262.89 158.75 0)
+      (effects (font (size 1.27 1.27)) hide)
+    )
+    (pin "1")
+  )
   (symbol (lib_id "power:GND") (at 59.69 184.15 0) (unit 1)
     (in_bom yes) (on_board yes) (fields_autoplaced)
@@
     )
     (property "Datasheet" "" (id 3) (at 228.6 62.23 0)
+      (effects (font (size 1.27 1.27)) hide)
+    )
+    (pin "1")
+  )
+  (symbol (lib_id "power:PWR_FLAG") (at 273.05 158.75 180) (unit 1)
+    (in_bom yes) (on_board yes) (fields_autoplaced)
+    (property "Reference" "#FLG02" (id 0) (at 273.05 160.655 0)
+      (effects (font (size 1.27 1.27)) hide)
+    )
+    (property "Value" "PWR_FLAG" (id 1) (at 273.05 163.83 0))
+    (property "Footprint" "" (id 2) (at 273.05 158.75 0)
+      (effects (font (size 1.27 1.27)) hide)
+    )
+    (property "Datasheet" "~" (id 3) (at 273.05 158.75 0)
       (effects (font (size 1.27 1.27)) hide)
     )
@@
     (pin "9")
   )
+  (symbol (lib_id "power:PWR_FLAG") (at 262.89 154.94 0) (unit 1)
+    (in_bom yes) (on_board yes) (fields_autoplaced)
+    (property "Reference" "#FLG01" (id 0) (at 262.89 153.035 0)
+      (effects (font (size 1.27 1.27)) hide)
+    )
+    (property "Value" "PWR_FLAG" (id 1) (at 262.89 149.86 0))
+    (property "Footprint" "" (id 2) (at 262.89 154.94 0)
+      (effects (font (size 1.27 1.27)) hide)
+    )
+    (property "Datasheet" "~" (id 3) (at 262.89 154.94 0)
+      (effects (font (size 1.27 1.27)) hide)
+    )
+    (pin "1")
+  )
   (symbol (lib_id "power:GND") (at 161.29 53.34 0) (unit 1)
     (in_bom yes) (on_board yes) (fields_autoplaced)
@@
     )
     (property "Datasheet" "" (id 3) (at 227.33 125.73 0)
+      (effects (font (size 1.27 1.27)) hide)
+    )
+    (pin "1")
+  )
+  (symbol (lib_id "power:+5V") (at 273.05 154.94 0) (unit 1)
+    (in_bom yes) (on_board yes)
+    (property "Reference" "#PWR06" (id 0) (at 273.05 158.75 0)
+      (effects (font (size 1.27 1.27)) hide)
+    )
+    (property "Value" "+5V" (id 1) (at 273.05 151.13 0))
+    (property "Footprint" "" (id 2) (at 273.05 154.94 0)
+      (effects (font (size 1.27 1.27)) hide)
+    )
+    (property "Datasheet" "" (id 3) (at 273.05 154.94 0)
       (effects (font (size 1.27 1.27)) hide)
     )
@@
   )
   (symbol_instances
+    (path "/c507f83d-cb5c-4edd-a401-1cdcab44c37b"
+      (reference "#FLG01") (unit 1) (value "PWR_FLAG") (footprint "")
+    )
+    (path "/3a597f40-d8e4-4b64-9092-5f5cfe33e399"
+      (reference "#FLG02") (unit 1) (value "PWR_FLAG") (footprint "")
+    )
     (path "/95513a1e-866d-4796-ba67-2729d6d9a203"
       (reference "#PWR01") (unit 1) (value "+5V") (footprint "")
@@
       (reference "#PWR04") (unit 1) (value "+5V") (footprint "")
     )
+    (path "/0ea5412c-cc52-4b0f-94f7-b24292ff04f3"
+      (reference "#PWR05") (unit 1) (value "GND") (footprint "")
+    )
+    (path "/fa7fbab3-4586-45b5-91f6-9e15c6c505fe"
+      (reference "#PWR06") (unit 1) (value "+5V") (footprint "")
+    )
     (path "/580d246c-7d7f-42d0-86df-37541ac0298d"
